File: KiCad/LDAD_ATOM _PRO _LCD _ABS_Enclosure_52x48.kicad_pcb (KiCad board)
At the start: 2 copper layers, 52.9 x 46.4 mm, 114 parts, among them CN3065_C2 4.7uF, CN3065_R1 1K8, CN3065_STDBY_LED1 LED, CN3965_C1 22uF, J1 TYPE-C-31-M-12, U1 MCP1525-TT, U2 ATSHA204A-MAHDA-T, U3 Battery_charger_CN3065_QFN8, U4 AHT20, U6 TEMT6000

Commit message: Add files via upload
Parts:
- added ATH20_C1: 100nF, Capacitor_SMD:C_0603_1608Metric, F.Cu at (217.4, 75.6)
- added IC_ENS1: ~, AeonLabs_Sensors:ENS160 Gas Semsor, B.Cu at (229.8, 77.5)
- added U5: BMP280, AeonLabs_Sensors:XDCR_BMP280, B.Cu at (229.8, 74.0)
- U2: footprint Package_SO:ATSHA204A Auth SOIC8 -> AeonLabs_IC:ATSHA204 UDFN-8 DFN200X300X60-9N
- moved U6 2.52 mm to (232.8, 75.6), turned to 90 degrees
- moved U2 1.95 mm to (217.2, 86.5)
- moved IMU1 0.23 mm to (221.8, 86.8)
Connections:
- ExtSW1 pad MP: GNDD -> (no net)
- ExtSWBAT_PLUG2 pad MP: GNDD -> (no net)
- I2C_PLUG1 pad MP: GNDD -> (no net)
- JICSP1 pad MP: GNDD -> (no net)
- PWR_PLUG1 pad MP: GNDD -> (no net)
Routing:
- net GNDD: track 135.9 -> 167.6 mm
- net 3V3: track 224.9 -> 248.7 mm, vias 18 -> 17
- net GPIO8_I2C_SDA: track 76.9 -> 87.0 mm, vias 5 -> 6
- net GPIO9_I2C_SCL: track 73.2 -> 80.8 mm, vias 5 -> 6
- net TEMT6000_IO33: track 98.6 -> 93.2 mm
- net (no net): track 2.74 -> 0.00 mm
Other:
- board text added: "12-Bit"
- board text added: "12-Bit Smart DAQ"
- board text added: "Environment Sensors"
- board text removed: "12-16Bit Smart DAQ"
- board text removed: "Luminosity Sensor"
- board text removed: "Sensor HT"
